Commit message: rviz sensor colour

File: urdf/sensor.urdf.xacro (robot description, xacro)
@@ -1,17 +1,87 @@
 <?xml version="1.0"?>
 <robot xmlns:xacro="http://www.ros.org/wiki/xacro" name="robot">
+    <material name="red">
+        <color rgba="1 0 0 1"/>
+    </material>
+    <material name="green">
+        <color rgba="0 1 0 1"/>
+    </material>
+    <material name="blue">
+        <color rgba="0 0 1 1"/>
+    </material>
+    <xacro:property name="lx" value="0.5"/>
+    <xacro:property name="ly" value="0.5"/>
+    <xacro:property name="lz" value="0.2"/>
+    <xacro:property name="t" value="0.005"/>
     <link name="sensor_link">
-        <visual>
-            <origin xyz="0.0 0.0 0.0"/>
+        <collision>
+            <origin xyz="0 0 0"/>
             <geometry>
-                <box size="0.3 0.3 0.15"/>
-            </geometry>
-        </visual>
-        <collision>
-            <origin xyz="0.0 0.0 0.0"/>
-            <geometry>
-                <box size="0.3 0.3 0.15"/>
+                <box size="${lx-2*t} ${ly-2*t} ${lz-2*t}"/>
             </geometry>
         </collision>
     </link>
+    <joint name="sensor_z_joint" type="fixed">
+        <parent link="sensor_link"/>
+        <child link="sensor_z"/>
+        <origin xyz="0 0 0"/>
+    </joint>
+    <link name="sensor_z">
+        <visual>
+            <origin xyz="0 0 ${lz/2 - t/2}"/>
+            <geometry>
+                <box size="${lx} ${ly} ${t}"/>
+            </geometry>
+            <material name="blue"/>
+        </visual>
+        <visual>
+            <origin xyz="0 0 ${-lz/2 + t/2}"/>
+            <geometry>
+                <box size="${lx} ${ly} ${t}"/>
+            </geometry>
+            <material name="blue"/>
+        </visual>
+    </link>
+    <joint name="sensor_y_join" type="fixed">
+        <parent link="sensor_link"/>
+        <child link="sensor_y"/>
+        <origin xyz="0 0 0"/>
+    </joint>
+    <link name="sensor_y">
+        <visual>
+            <origin xyz="0 ${ly/2 - t/2} 0"/>
+            <geometry>
+                <box size="${lx-2*t} ${t} ${lz-2*t}"/>
+            </geometry>
+            <material name="green"/>
+        </visual>
+        <visual>
+            <origin xyz="0 ${-ly/2 + t/2} 0"/>
+            <geometry>
+                <box size="${lx-2*t} ${t} ${lz-2*t}"/>
+            </geometry>
+            <material name="green"/>
+        </visual>
+    </link>
+    <joint name="sensor_x_join" type="fixed">
+        <parent link="sensor_link"/>
+        <child link="sensor_x"/>
+        <origin xyz="0 0 0"/>
+    </joint>
+    <link name="sensor_x">
+        <visual>
+            <origin xyz="${lx/2 - t/2} 0 0"/>
+            <geometry>
+                <box size="${t} ${ly-2*t} ${lz-2*t}"/>
+            </geometry>
+            <material name="red"/>
+        </visual>
+        <visual>
+            <origin xyz="${-lx/2 + t/2} 0 0"/>
+            <geometry>
+                <box size="${t} ${ly-2*t} ${lz-2*t}"/>
+            </geometry>
+            <material name="red"/>
+        </visual>
+    </link>
 </robot>
